File: proteus.kicad_sch (KiCad schematic)
At the start: 29 parts, among them J1 Conn_01x01, J15 Sicma_56, J2 Conn_01x01, J3 Conn_01x01, J4 Conn_01x03, J5 Conn_01x05, J6 Conn_02x04_Counter_Clockwise, J9 Conn_01x04

Commit message: USB jack, parts and LCSC numbers, headphone jack
Parts:
- C1: LCSC N/A -> C106564
Changed lines of the file:
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@@
       (effects (font (size 1.27 1.27)) hide)
     )
-    (property "LCSC" "N/A" (at 272.415 90.17 0)
+    (property "LCSC" "C106564" (at 272.415 90.17 0)
       (effects (font (size 1.27 1.27)) hide)
     )
