File: lowside_uln2003.kicad_sch (KiCad schematic)
At the start: 5 parts, among them U12 TBD62083AFWG

Commit message: update
Parts:
- added U15 (x8): 2k7, Resistor_SMD:R_0805_2012Metric, symbol Device:R
- added U31 (x8): RED, LED_SMD:LED_0805_2012Metric, symbol Device:LED
Connections:
- net 12V: now also U15.2, U15.2, U15.2, U15.2, U15.2, U15.2, U15.2, U15.2
- net OUT1: now also U31.1 (K)
- net OUT2: now also U31.1 (K)
- net OUT3: now also U31.1 (K)
- net OUT4: now also U31.1 (K)
- net OUT5: now also U31.1 (K)
- net OUT6: now also U31.1 (K)
- net OUT7: now also U31.1 (K)
- net OUT8: now also U31.1 (K)
- new net: U15.1, U31.2 (A) (x8)

Commit message: USB jack, parts and LCSC numbers, headphone jack
Parts:
- U15: footprint Resistor_SMD:R_0805_2012Metric -> Resistor_SMD:R_0402_1005Metric; LCSC (none) -> C138017
- U31: footprint LED_SMD:LED_0805_2012Metric -> LED_SMD:LED_0603_1608Metric; LCSC (none) -> C84263
Changed lines of the file:
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@@
       (effects (font (size 1.27 1.27)))
     )
-    (property "Footprint" "LED_SMD:LED_0805_2012Metric" (at 212.09 82.55 0)
+    (property "Footprint" "LED_SMD:LED_0603_1608Metric" (at 212.09 82.55 0)
       (effects (font (size 1.27 1.27)) hide)
     )
     (property "Datasheet" "" (at 212.09 82.55 0)
       (effects (font (size 1.27 1.27)))
+    )
+    (property "LCSC" "C84263" (at 212.09 82.55 0)
+      (effects (font (size 1.27 1.27)) hide)
     )
     (pin "1")
@@
       (effects (font (size 1.27 1.27)))
     )
-    (property "Footprint" "Resistor_SMD:R_0805_2012Metric" (at 200.66 118.872 90)
+    (property "Footprint" "Resistor_SMD:R_0402_1005Metric" (at 200.66 118.872 90)
       (effects (font (size 1.27 1.27)) hide)
     )
     (property "Datasheet" "" (at 200.66 120.65 0)
       (effects (font (size 1.27 1.27)))
+    )
+    (property "LCSC" "C138017" (at 200.66 120.65 90)
+      (effects (font (size 1.27 1.27)) hide)
     )
     (pin "1")
@@
       (effects (font (size 1.27 1.27)))
     )
-    (property "Footprint" "Resistor_SMD:R_0805_2012Metric" (at 200.66 65.532 90)
+    (property "Footprint" "Resistor_SMD:R_0402_1005Metric" (at 200.66 65.532 90)
       (effects (font (size 1.27 1.27)) hide)
     )
@@
       (effects (font (size 1.27 1.27)))
     )
+    (property "LCSC" "C138017" (at 200.66 67.31 90)
+      (effects (font (size 1.27 1.27)) hide)
+    )
     (pin "1")
     (pin "2")
@@
       (effects (font (size 1.27 1.27)))
     )
-    (property "Footprint" "Resistor_SMD:R_0805_2012Metric" (at 200.66 96.012 90)
+    (property "Footprint" "Resistor_SMD:R_0402_1005Metric" (at 200.66 96.012 90)
       (effects (font (size 1.27 1.27)) hide)
     )
@@
       (effects (font (size 1.27 1.27)))
     )
+    (property "LCSC" "C138017" (at 200.66 97.79 90)
+      (effects (font (size 1.27 1.27)) hide)
+    )
     (pin "1")
     (pin "2")
@@
       (effects (font (size 1.27 1.27)))
     )
-    (property "Footprint" "LED_SMD:LED_0805_2012Metric" (at 212.09 120.65 0)
+    (property "Footprint" "LED_SMD:LED_0603_1608Metric" (at 212.09 120.65 0)
       (effects (font (size 1.27 1.27)) hide)
     )
@@
       (effects (font (size 1.27 1.27)))
     )
+    (property "LCSC" "C84263" (at 212.09 120.65 0)
+      (effects (font (size 1.27 1.27)) hide)
+    )
     (pin "1")
     (pin "2")
@@
       (effects (font (size 1.27 1.27)))
     )
-    (property "Footprint" "Resistor_SMD:R_0805_2012Metric" (at 200.66 80.772 90)
+    (property "Footprint" "Resistor_SMD:R_0402_1005Metric" (at 200.66 80.772 90)
       (effects (font (size 1.27 1.27)) hide)
     )
@@
       (effects (font (size 1.27 1.27)))
     )
+    (property "LCSC" "C138017" (at 200.66 82.55 90)
+      (effects (font (size 1.27 1.27)) hide)
+    )
     (pin "1")
     (pin "2")
@@
       (effects (font (size 1.27 1.27)))
     )
-    (property "Footprint" "LED_SMD:LED_0805_2012Metric" (at 212.09 105.41 0)
+    (property "Footprint" "LED_SMD:LED_0603_1608Metric" (at 212.09 105.41 0)
       (effects (font (size 1.27 1.27)) hide)
     )
@@
       (effects (font (size 1.27 1.27)))
     )
+    (property "LCSC" "C84263" (at 212.09 105.41 0)
+      (effects (font (size 1.27 1.27)) hide)
+    )
     (pin "1")
     (pin "2")
@@
       (effects (font (size 1.27 1.27)))
     )
-    (property "Footprint" "LED_SMD:LED_0805_2012Metric" (at 212.09 97.79 0)
+    (property "Footprint" "LED_SMD:LED_0603_1608Metric" (at 212.09 97.79 0)
       (effects (font (size 1.27 1.27)) hide)
     )
@@
       (effects (font (size 1.27 1.27)))
     )
+    (property "LCSC" "C84263" (at 212.09 97.79 0)
+      (effects (font (size 1.27 1.27)) hide)
+    )
     (pin "1")
     (pin "2")
@@
       (effects (font (size 1.27 1.27)))
     )
-    (property "Footprint" "LED_SMD:LED_0805_2012Metric" (at 212.09 74.93 0)
+    (property "Footprint" "LED_SMD:LED_0603_1608Metric" (at 212.09 74.93 0)
       (effects (font (size 1.27 1.27)) hide)
     )
@@
       (effects (font (size 1.27 1.27)))
     )
+    (property "LCSC" "C84263" (at 212.09 74.93 0)
+      (effects (font (size 1.27 1.27)) hide)
+    )
     (pin "1")
     (pin "2")
@@
       (effects (font (size 1.27 1.27)))
     )
-    (property "Footprint" "LED_SMD:LED_0805_2012Metric" (at 212.09 113.03 0)
+    (property "Footprint" "LED_SMD:LED_0603_1608Metric" (at 212.09 113.03 0)
       (effects (font (size 1.27 1.27)) hide)
     )
@@
       (effects (font (size 1.27 1.27)))
     )
+    (property "LCSC" "C84263" (at 212.09 113.03 0)
+      (effects (font (size 1.27 1.27)) hide)
+    )
     (pin "1")
     (pin "2")
@@
       (effects (font (size 1.27 1.27)))
     )
-    (property "Footprint" "Resistor_SMD:R_0805_2012Metric" (at 200.66 88.392 90)
+    (property "Footprint" "Resistor_SMD:R_0402_1005Metric" (at 200.66 88.392 90)
       (effects (font (size 1.27 1.27)) hide)
     )
@@
       (effects (font (size 1.27 1.27)))
     )
+    (property "LCSC" "C138017" (at 200.66 90.17 90)
+      (effects (font (size 1.27 1.27)) hide)
+    )
     (pin "1")
     (pin "2")
@@
       (effects (font (size 1.27 1.27)))
     )
-    (property "Footprint" "LED_SMD:LED_0805_2012Metric" (at 212.09 90.17 0)
+    (property "Footprint" "LED_SMD:LED_0603_1608Metric" (at 212.09 90.17 0)
       (effects (font (size 1.27 1.27)) hide)
     )
@@
       (effects (font (size 1.27 1.27)))
     )
+    (property "LCSC" "C84263" (at 212.09 90.17 0)
+      (effects (font (size 1.27 1.27)) hide)
+    )
     (pin "1")
     (pin "2")
@@
       (effects (font (size 1.27 1.27)))
     )
-    (property "Footprint" "LED_SMD:LED_0805_2012Metric" (at 212.09 67.31 0)
+    (property "Footprint" "LED_SMD:LED_0603_1608Metric" (at 212.09 67.31 0)
       (effects (font (size 1.27 1.27)) hide)
     )
     (property "Datasheet" "" (at 212.09 67.31 0)
       (effects (font (size 1.27 1.27)))
+    )
+    (property "LCSC" "C84263" (at 212.09 67.31 0)
+      (effects (font (size 1.27 1.27)) hide)
     )
     (pin "1")
@@
       (effects (font (size 1.27 1.27)))
     )
-    (property "Footprint" "Resistor_SMD:R_0805_2012Metric" (at 200.66 73.152 90)
+    (property "Footprint" "Resistor_SMD:R_0402_1005Metric" (at 200.66 73.152 90)
       (effects (font (size 1.27 1.27)) hide)
     )
     (property "Datasheet" "" (at 200.66 74.93 0)
       (effects (font (size 1.27 1.27)))
+    )
+    (property "LCSC" "C138017" (at 200.66 74.93 90)
+      (effects (font (size 1.27 1.27)) hide)
     )
     (pin "1")
@@
       (effects (font (size 1.27 1.27)))
     )
-    (property "Footprint" "Resistor_SMD:R_0805_2012Metric" (at 200.66 103.632 90)
+    (property "Footprint" "Resistor_SMD:R_0402_1005Metric" (at 200.66 103.632 90)
       (effects (font (size 1.27 1.27)) hide)
     )
@@
       (effects (font (size 1.27 1.27)))
     )
+    (property "LCSC" "C138017" (at 200.66 105.41 90)
+      (effects (font (size 1.27 1.27)) hide)
+    )
     (pin "1")
     (pin "2")
@@
       (effects (font (size 1.27 1.27)))
     )
-    (property "Footprint" "Resistor_SMD:R_0805_2012Metric" (at 200.66 111.252 90)
+    (property "Footprint" "Resistor_SMD:R_0402_1005Metric" (at 200.66 111.252 90)
       (effects (font (size 1.27 1.27)) hide)
     )
@@
       (effects (font (size 1.27 1.27)))
     )
-    (pin "1")
+    (property "LCSC" "C138017" (at 200.66 113.03 90)
+      (effects (font (size 1.27 1.27)) hide)
+    )
+    (pin "1")

Commit message: Add Stepper, fix Connector, add Testpoints, several changes
Parts:
- U31: LCSC C84263 -> C2286
Changed lines of the file:
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@@
       (effects (font (size 1.27 1.27)))
     )
-    (property "LCSC" "C84263" (at 212.09 82.55 0)
+    (property "LCSC" "C2286" (at 212.09 82.55 0)
       (effects (font (size 1.27 1.27)) hide)
     )
@@
       (effects (font (size 1.27 1.27)))
     )
-    (property "LCSC" "C84263" (at 212.09 120.65 0)
+    (property "LCSC" "C2286" (at 212.09 120.65 0)
       (effects (font (size 1.27 1.27)) hide)
     )
@@
       (effects (font (size 1.27 1.27)))
     )
-    (property "LCSC" "C84263" (at 212.09 105.41 0)
+    (property "LCSC" "C2286" (at 212.09 105.41 0)
       (effects (font (size 1.27 1.27)) hide)
     )
@@
       (effects (font (size 1.27 1.27)))
     )
-    (property "LCSC" "C84263" (at 212.09 97.79 0)
+    (property "LCSC" "C2286" (at 212.09 97.79 0)
       (effects (font (size 1.27 1.27)) hide)
     )
@@
       (effects (font (size 1.27 1.27)))
     )
-    (property "LCSC" "C84263" (at 212.09 74.93 0)
+    (property "LCSC" "C2286" (at 212.09 74.93 0)
       (effects (font (size 1.27 1.27)) hide)
     )
@@
       (effects (font (size 1.27 1.27)))
     )
-    (property "LCSC" "C84263" (at 212.09 113.03 0)
+    (property "LCSC" "C2286" (at 212.09 113.03 0)
       (effects (font (size 1.27 1.27)) hide)
     )
@@
       (effects (font (size 1.27 1.27)))
     )
-    (property "LCSC" "C84263" (at 212.09 90.17 0)
+    (property "LCSC" "C2286" (at 212.09 90.17 0)
       (effects (font (size 1.27 1.27)) hide)
     )
@@
       (effects (font (size 1.27 1.27)))
     )
-    (property "LCSC" "C84263" (at 212.09 67.31 0)
-      (effects (font (size 1.27 1.27)) hide)
-    )
+    (property "LCSC" "C2286" (at 212.09 67.31 0)
+      (effects (font (size 1.27 1.27)) hide)
+    )
