File: psu.kicad_sch (KiCad schematic)
At the start: 49 parts, among them U1 TLS115, U3 LMR14020, U39 1N4148WS, U4 TJA1051T-3, U5 TJA1051T-3, U6 AMS1117-3.3

Commit message: Production optimizations, voltage superv, etb sv conn
Parts:
- C6: JLCPosOffset (none) -> 1.75,0
- D19, D5: LCSC C151281 -> C406701; LCSC_ext C406701 -> C151281
Changed lines of the file:
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@@
       (effects (font (size 1.27 1.27)) hide)
     )
-    (property "LCSC" "C151281" (at 29.21 34.29 0)
-      (effects (font (size 1.27 1.27)) hide)
-    )
-    (property "LCSC_ext" "C406701" (at 29.21 34.29 0)
+    (property "LCSC" "C406701" (at 29.21 34.29 0)
+      (effects (font (size 1.27 1.27)) hide)
+    )
+    (property "LCSC_ext" "C151281" (at 29.21 34.29 0)
       (effects (font (size 1.27 1.27)) hide)
     )
@@
     )
     (property "LCSC" "C106564" (at 99.695 35.56 0)
+      (effects (font (size 1.27 1.27)) hide)
+    )
+    (property "JLCPosOffset" "1.75,0" (at 99.695 35.56 0)
       (effects (font (size 1.27 1.27)) hide)
     )
@@
       (effects (font (size 1.27 1.27)) hide)
     )
-    (property "LCSC" "C151281" (at 29.21 64.135 0)
-      (effects (font (size 1.27 1.27)) hide)
-    )
-    (property "LCSC_ext" "C406701" (at 29.21 64.135 0)
-      (effects (font (size 1.27 1.27)) hide)
-    )
+    (property "LCSC" "C406701" (at 29.21 64.135 0)
+      (effects (font (size 1.27 1.27)) hide)
+    )
+    (property "LCSC_ext" "C151281" (at 29.21 64.135 0)
+      (effects (font (size 1.27 1.27)) hide)
+    )
