File: etbsupervisor.kicad_sch (KiCad schematic)
At the start: 5 parts, among them J18 Conn_02x04_Counter_Clockwise

Commit message: Optimize
Parts:
- removed D18: SRV05-4, Package_TO_SOT_SMD:SOT-23-6, symbol Power_Protection:SRV05-4
Connections:
- net 12V_DIVIDED renamed SRV05-4
- no-connect marks 3 -> 0
Other:
- note added: "Protection shared with mcu"
- note removed: "1.3V @ 12V"
Changed lines of the file:
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@@
   (junction (at 173.99 83.185) (diameter 0) (color 0 0 0 0)
   )
+  (junction (at 186.055 83.185) (diameter 0) (color 0 0 0 0)
+  )
   (junction (at 163.195 83.185) (diameter 0) (color 0 0 0 0)
   )
-  (no_connect (at 202.565 88.265))
-  (no_connect (at 227.965 83.185))
-  (no_connect (at 227.965 88.265))
   (wire (pts (xy 87.63 97.155) (xy 86.995 97.155))
     (stroke (width 0) (type default))
@@
     (stroke (width 0) (type default))
   )
-  (wire (pts (xy 173.99 83.185) (xy 202.565 83.185))
+  (wire (pts (xy 173.99 83.185) (xy 186.055 83.185))
     (stroke (width 0) (type default))
   )
@@
     (stroke (width 0) (type default))
   )
+  (wire (pts (xy 186.055 83.185) (xy 202.565 83.185))
+    (stroke (width 0) (type default))
+  )
   (polyline (pts (xy 127 66.04) (xy 231.14 66.04))
     (stroke (width 0) (type default))
@@
     (stroke (width 0) (type default))
   )
+  (wire (pts (xy 187.96 86.36) (xy 186.055 86.36))
+    (stroke (width 0) (type default))
+  )
   (wire (pts (xy 80.645 94.615) (xy 87.63 94.615))
     (stroke (width 0) (type default))
@@
     (stroke (width 0) (type default))
   )
+  (wire (pts (xy 186.055 86.36) (xy 186.055 83.185))
+    (stroke (width 0) (type default))
+  )
   (wire (pts (xy 100.33 84.455) (xy 106.045 84.455))
     (stroke (width 0) (type default))
@@
     (stroke (width 0) (type default))
     (fill (type none))
+  )
+  (text "Protection shared with mcu" (at 185.42 88.9 0)
+    (effects (font (size 1.27 1.27)) (justify left bottom))
   )
   (text "External ETB Supervisor" (at 68.58 69.215 0)
     (effects (font (size 1.27 1.27)) (justify left bottom))
   )
-  (text "1.3V @ 12V" (at 180.34 73.66 0)
-    (effects (font (size 1.27 1.27)) (justify left bottom))
-  )
   (text "12V Sense Divider" (at 128.905 69.215 0)
     (effects (font (size 1.27 1.27)) (justify left bottom))
@@
     (effects (font (size 1.27 1.27)) (justify left))
   )
+  (hierarchical_label "SRV05-4" (shape output) (at 187.96 86.36 0) (fields_autoplaced)
+    (effects (font (size 1.27 1.27)) (justify left))
+  )
   (hierarchical_label "5V_SENSOR_S" (shape input) (at 106.045 86.995 0) (fields_autoplaced)
     (effects (font (size 1.27 1.27)) (justify left))
@@
         (path "/d9116601-cae2-4199-827b-70fa136aae51/de20b32b-d448-449a-9643-91f8f61343d8"
           (reference "#PWR0313") (unit 1)
-        )
-      )
-    )
-  )
-  (symbol (lib_id "proteus-rescue:+3.3V-power") (at 215.265 73.025 0) (unit 1)
-    (in_bom yes) (on_board yes) (dnp no)
-    (property "Reference" "#PWR0227" (at 215.265 76.835 0)
-      (effects (font (size 1.27 1.27)) hide)
-    )
-    (property "Value" "+3.3V" (at 215.646 68.6308 0)
-      (effects (font (size 1.27 1.27)))
-    )
-    (property "Footprint" "" (at 215.265 73.025 0)
-      (effects (font (size 1.27 1.27)) hide)
-    )
-    (property "Datasheet" "" (at 215.265 73.025 0)
-      (effects (font (size 1.27 1.27)) hide)
-    )
-    (pin "1")
-    (instances
-      (project "proteus"
-        (path "/d9116601-cae2-4199-827b-70fa136aae51/00000000-0000-0000-0000-00005d99e6ee"
-          (reference "#PWR0227") (unit 1)
-        )
-        (path "/d9116601-cae2-4199-827b-70fa136aae51/de20b32b-d448-449a-9643-91f8f61343d8"
-          (reference "#PWR0314") (unit 1)
         )
       )
@@
         )
       )
-    )
-  )
-  (symbol (lib_id "Power_Protection:SRV05-4") (at 215.265 85.725 0) (unit 1)
-    (in_bom yes) (on_board yes) (dnp no)
-    (property "Reference" "D18" (at 209.55 73.66 0)
-      (effects (font (size 1.27 1.27)))
-    )
-    (property "Value" "SRV05-4" (at 222.25 73.66 0)
-      (effects (font (size 1.27 1.27)))
-    )
-    (property "Footprint" "Package_TO_SOT_SMD:SOT-23-6" (at 233.045 97.155 0)
-      (effects (font (size 1.27 1.27)) hide)
-    )
-    (property "Datasheet" "http://www.onsemi.com/pub/Collateral/SRV05-4-D.PDF" (at 215.265 85.725 0)
-      (effects (font (size 1.27 1.27)) hide)
-    )
-    (property "LCSC" "C85364" (at 215.265 85.725 0)
-      (effects (font (size 1.27 1.27)) hide)
-    )
-    (property "LCSC_ext" "0" (at 215.265 85.725 0)
-      (effects (font (size 1.27 1.27)) hide)
-    )
-    (pin "1")
-    (pin "2")
-    (pin "3")
-    (pin "4")
-    (pin "5")
-    (pin "6")
-    (instances
-      (project "proteus"
-        (path "/d9116601-cae2-4199-827b-70fa136aae51/00000000-0000-0000-0000-00005d99e6ee"
-          (reference "D18") (unit 1)
-        )
-        (path "/d9116601-cae2-4199-827b-70fa136aae51/de20b32b-d448-449a-9643-91f8f61343d8"
-          (reference "D25") (unit 1)
-        )
-      )
-    )
-  )
-  (symbol (lib_id "power:GND") (at 215.265 98.425 0) (unit 1)
-    (in_bom yes) (on_board yes) (dnp no)
-    (property "Reference" "#PWR0228" (at 215.265 104.775 0)
-      (effects (font (size 1.27 1.27)) hide)
-    )
-    (property "Value" "GND" (at 215.392 102.8192 0)
-      (effects (font (size 1.27 1.27)))
-    )
-    (property "Footprint" "" (at 215.265 98.425 0)
-      (effects (font (size 1.27 1.27)) hide)
-    )
-    (property "Datasheet" "" (at 215.265 98.425 0)
-      (effects (font (size 1.27 1.27)) hide)
-    )
-    (pin "1")
-    (instances
-      (project "proteus"
-        (path "/d9116601-cae2-4199-827b-70fa136aae51/00000000-0000-0000-0000-00005d99e6ee"
-          (reference "#PWR0228") (unit 1)
-        )
-        (path "/d9116601-cae2-4199-827b-70fa136aae51/de20b32b-d448-449a-9643-91f8f61343d8"
-          (reference "#PWR0315") (unit 1)
-        )
-      )
